Commit message: Update mini_pupper code

File: mini_pupper_description/urdf/mini_pupper_2/mini_pupper_description.urdf.xacro (robot description, xacro)
@@ -24,14 +24,21 @@
       <origin xyz="0 0 0" rpy="0 0 0"/>
       <geometry>
-        <mesh filename="file://$(find mini_pupper_description)/meshes/mini_pupper_2/base_link.stl" scale="1 1 1"/>
-      </geometry>
-      <material name="opaque252525"/>
-    </visual>
-    <collision>
-      <origin xyz="0 0 0" rpy="0 0 0"/>
-      <geometry>
-        <mesh filename="file://$(find mini_pupper_description)/meshes/mini_pupper_2/base_link.stl" scale="1 1 1"/>
-      </geometry>
-    </collision>
+        <mesh filename="package://mini_pupper_description/meshes/mini_pupper_2/base_link_black.dae" scale="1 1 1"/>
+      </geometry>
+    </visual>
+    <collision>
+      <origin xyz="0 0 0" rpy="0 0 0"/>
+      <geometry>
+        <mesh filename="package://mini_pupper_description/meshes/mini_pupper_2/base_link.stl" scale="1 1 1"/>
+      </geometry>
+    </collision>
+  </link>
+  <link name="display_link">
+    <visual>
+      <origin xyz="0 0 0" rpy="0 0 0"/>
+      <geometry>
+        <mesh filename="package://mini_pupper_description/meshes/mini_pupper_2/displayscreen.dae" scale="1 1 1"/>
+      </geometry>
+    </visual>
   </link>
   <link name="base_inertia">
@@ -51,12 +58,11 @@
       <origin xyz="0 0 0" rpy="0 0 0"/>
       <geometry>
-        <mesh filename="file://$(find mini_pupper_description)/meshes/mini_pupper_2/lf1.stl" scale="1 1 1"/>
-      </geometry>
-      <material name="opaque666666"/>
-    </visual>
-    <collision>
-      <origin xyz="0 0 0" rpy="0 0 0"/>
-      <geometry>
-        <mesh filename="file://$(find mini_pupper_description)/meshes/mini_pupper_2/lf1.stl" scale="1 1 1"/>
+        <mesh filename="package://mini_pupper_description/meshes/mini_pupper_2/lf1_black.dae" scale="1 1 1"/>
+      </geometry>
+    </visual>
+    <collision>
+      <origin xyz="0 0 0" rpy="0 0 0"/>
+      <geometry>
+        <mesh filename="package://mini_pupper_description/meshes/mini_pupper_2/lf1.stl" scale="1 1 1"/>
       </geometry>
     </collision>
@@ -71,12 +77,11 @@
       <origin xyz="0 0 0" rpy="0 0 0"/>
       <geometry>
-        <mesh filename="file://$(find mini_pupper_description)/meshes/mini_pupper_2/lf2.stl" scale="1 1 1"/>
-      </geometry>
-      <material name="opaque636363"/>
-    </visual>
-    <collision>
-      <origin xyz="0 0 0" rpy="0 0 0"/>
-      <geometry>
-        <mesh filename="file://$(find mini_pupper_description)/meshes/mini_pupper_2/lf2.stl" scale="1 1 1"/>
+        <mesh filename="package://mini_pupper_description/meshes/mini_pupper_2/lf2.dae" scale="1 1 1"/>
+      </geometry>
+    </visual>
+    <collision>
+      <origin xyz="0 0 0" rpy="0 0 0"/>
+      <geometry>
+        <mesh filename="package://mini_pupper_description/meshes/mini_pupper_2/lf2.stl" scale="1 1 1"/>
       </geometry>
     </collision>
@@ -91,12 +96,11 @@
       <origin xyz="0 0 0" rpy="0 0 0"/>
       <geometry>
-        <mesh filename="file://$(find mini_pupper_description)/meshes/mini_pupper_2/lf3.stl" scale="1 1 1"/>
-      </geometry>
-      <material name="opaque252525"/>
-    </visual>
-    <collision>
-      <origin xyz="0 0 0" rpy="0 0 0"/>
-      <geometry>
-        <mesh filename="file://$(find mini_pupper_description)/meshes/mini_pupper_2/lf3.stl" scale="1 1 1"/>
+        <mesh filename="package://mini_pupper_description/meshes/mini_pupper_2/lf3.dae" scale="1 1 1"/>
+      </geometry>
+    </visual>
+    <collision>
+      <origin xyz="0 0 0" rpy="0 0 0"/>
+      <geometry>
+        <mesh filename="package://mini_pupper_description/meshes/mini_pupper_2/lf3.stl" scale="1 1 1"/>
       </geometry>
     </collision>
@@ -111,12 +115,11 @@
       <origin xyz="0 0 0" rpy="0 0 0"/>
       <geometry>
-        <mesh filename="file://$(find mini_pupper_description)/meshes/mini_pupper_2/rf1.stl" scale="1 1 1"/>
-      </geometry>
-      <material name="opaque666666"/>
-    </visual>
-    <collision>
-      <origin xyz="0 0 0" rpy="0 0 0"/>
-      <geometry>
-        <mesh filename="file://$(find mini_pupper_description)/meshes/mini_pupper_2/rf1.stl" scale="1 1 1"/>
+        <mesh filename="package://mini_pupper_description/meshes/mini_pupper_2/rf1.dae" scale="1 1 1"/>
+      </geometry>
+    </visual>
+    <collision>
+      <origin xyz="0 0 0" rpy="0 0 0"/>
+      <geometry>
+        <mesh filename="package://mini_pupper_description/meshes/mini_pupper_2/rf1.stl" scale="1 1 1"/>
       </geometry>
     </collision>
@@ -131,12 +134,11 @@
       <origin xyz="0 0 0" rpy="0 0 0"/>
       <geometry>
-        <mesh filename="file://$(find mini_pupper_description)/meshes/mini_pupper_2/rf2.stl" scale="1 1 1"/>
-      </geometry>
-      <material name="opaque636363"/>
-    </visual>
-    <collision>
-      <origin xyz="0 0 0" rpy="0 0 0"/>
-      <geometry>
-        <mesh filename="file://$(find mini_pupper_description)/meshes/mini_pupper_2/rf2.stl" scale="1 1 1"/>
+        <mesh filename="package://mini_pupper_description/meshes/mini_pupper_2/rf2.dae" scale="1 1 1"/>
+      </geometry>
+    </visual>
+    <collision>
+      <origin xyz="0 0 0" rpy="0 0 0"/>
+      <geometry>
+        <mesh filename="package://mini_pupper_description/meshes/mini_pupper_2/rf2.stl" scale="1 1 1"/>
       </geometry>
     </collision>
@@ -151,12 +153,11 @@
       <origin xyz="0 0 0" rpy="0 0 0"/>
       <geometry>
-        <mesh filename="file://$(find mini_pupper_description)/meshes/mini_pupper_2/rf3.stl" scale="1 1 1"/>
-      </geometry>
-      <material name="opaque252525"/>
-    </visual>
-    <collision>
-      <origin xyz="0 0 0" rpy="0 0 0"/>
-      <geometry>
-        <mesh filename="file://$(find mini_pupper_description)/meshes/mini_pupper_2/rf3.stl" scale="1 1 1"/>
+        <mesh filename="package://mini_pupper_description/meshes/mini_pupper_2/rf3_black.dae" scale="1 1 1"/>
+      </geometry>
+    </visual>
+    <collision>
+      <origin xyz="0 0 0" rpy="0 0 0"/>
+      <geometry>
+        <mesh filename="package://mini_pupper_description/meshes/mini_pupper_2/rf3.stl" scale="1 1 1"/>
       </geometry>
     </collision>
@@ -171,12 +172,11 @@
       <origin xyz="0 0 0" rpy="0 0 0"/>
       <geometry>
-        <mesh filename="file://$(find mini_pupper_description)/meshes/mini_pupper_2/rb1.stl" scale="1 1 1"/>
-      </geometry>
-      <material name="opaque666666"/>
-    </visual>
-    <collision>
-      <origin xyz="0 0 0" rpy="0 0 0"/>
-      <geometry>
-        <mesh filename="file://$(find mini_pupper_description)/meshes/mini_pupper_2/rb1.stl" scale="1 1 1"/>
+        <mesh filename="package://mini_pupper_description/meshes/mini_pupper_2/rb1.dae" scale="1 1 1"/>
+      </geometry>
+    </visual>
+    <collision>
+      <origin xyz="0 0 0" rpy="0 0 0"/>
+      <geometry>
+        <mesh filename="package://mini_pupper_description/meshes/mini_pupper_2/rb1.stl" scale="1 1 1"/>
       </geometry>
     </collision>
@@ -191,12 +191,11 @@
       <origin xyz="0 0 0" rpy="0 0 0"/>
       <geometry>
-        <mesh filename="file://$(find mini_pupper_description)/meshes/mini_pupper_2/rb2.stl" scale="1 1 1"/>
-      </geometry>
-      <material name="opaque636363"/>
-    </visual>
-    <collision>
-      <origin xyz="0 0 0" rpy="0 0 0"/>
-      <geometry>
-        <mesh filename="file://$(find mini_pupper_description)/meshes/mini_pupper_2/rb2.stl" scale="1 1 1"/>
+        <mesh filename="package://mini_pupper_description/meshes/mini_pupper_2/rb2.dae" scale="1 1 1"/>
+      </geometry>
+    </visual>
+    <collision>
+      <origin xyz="0 0 0" rpy="0 0 0"/>
+      <geometry>
+        <mesh filename="package://mini_pupper_description/meshes/mini_pupper_2/rb2.stl" scale="1 1 1"/>
       </geometry>
     </collision>
@@ -211,12 +210,11 @@
       <origin xyz="0 0 0" rpy="0 0 0"/>
       <geometry>
-        <mesh filename="file://$(find mini_pupper_description)/meshes/mini_pupper_2/rb3.stl" scale="1 1 1"/>
-      </geometry>
-      <material name="opaque252525"/>
-    </visual>
-    <collision>
-      <origin xyz="0 0 0" rpy="0 0 0"/>
-      <geometry>
-        <mesh filename="file://$(find mini_pupper_description)/meshes/mini_pupper_2/rb3.stl" scale="1 1 1"/>
+        <mesh filename="package://mini_pupper_description/meshes/mini_pupper_2/rb3.dae" scale="1 1 1"/>
+      </geometry>
+    </visual>
+    <collision>
+      <origin xyz="0 0 0" rpy="0 0 0"/>
+      <geometry>
+        <mesh filename="package://mini_pupper_description/meshes/mini_pupper_2/rb3.stl" scale="1 1 1"/>
       </geometry>
     </collision>
@@ -231,12 +229,11 @@
       <origin xyz="0 0 0" rpy="0 0 0"/>
       <geometry>
-        <mesh filename="file://$(find mini_pupper_description)/meshes/mini_pupper_2/lb1.stl" scale="1 1 1"/>
-      </geometry>
-      <material name="opaque666666"/>
-    </visual>
-    <collision>
-      <origin xyz="0 0 0" rpy="0 0 0"/>
-      <geometry>
-        <mesh filename="file://$(find mini_pupper_description)/meshes/mini_pupper_2/lb1.stl" scale="1 1 1"/>
+        <mesh filename="package://mini_pupper_description/meshes/mini_pupper_2/lb1.dae" scale="1 1 1"/>
+      </geometry>
+    </visual>
+    <collision>
+      <origin xyz="0 0 0" rpy="0 0 0"/>
+      <geometry>
+        <mesh filename="package://mini_pupper_description/meshes/mini_pupper_2/lb1.stl" scale="1 1 1"/>
       </geometry>
     </collision>
@@ -251,12 +248,11 @@
       <origin xyz="0 0 0" rpy="0 0 0"/>
       <geometry>
-        <mesh filename="file://$(find mini_pupper_description)/meshes/mini_pupper_2/lb2.stl" scale="1 1 1"/>
-      </geometry>
-      <material name="opaque636363"/>
-    </visual>
-    <collision>
-      <origin xyz="0 0 0" rpy="0 0 0"/>
-      <geometry>
-        <mesh filename="file://$(find mini_pupper_description)/meshes/mini_pupper_2/lb2.stl" scale="1 1 1"/>
+        <mesh filename="package://mini_pupper_description/meshes/mini_pupper_2/lb2.dae" scale="1 1 1"/>
+      </geometry>
+    </visual>
+    <collision>
+      <origin xyz="0 0 0" rpy="0 0 0"/>
+      <geometry>
+        <mesh filename="package://mini_pupper_description/meshes/mini_pupper_2/lb2.stl" scale="1 1 1"/>
       </geometry>
     </collision>
@@ -271,12 +267,11 @@
       <origin xyz="0 0 0" rpy="0 0 0"/>
       <geometry>
-        <mesh filename="file://$(find mini_pupper_description)/meshes/mini_pupper_2/lb3.stl" scale="1 1 1"/>
-      </geometry>
-      <material name="opaque252525"/>
-    </visual>
-    <collision>
-      <origin xyz="0 0 0" rpy="0 0 0"/>
-      <geometry>
-        <mesh filename="file://$(find mini_pupper_description)/meshes/mini_pupper_2/lb3.stl" scale="1 1 1"/>
+        <mesh filename="package://mini_pupper_description/meshes/mini_pupper_2/lb3.dae" scale="1 1 1"/>
+      </geometry>
+    </visual>
+    <collision>
+      <origin xyz="0 0 0" rpy="0 0 0"/>
+      <geometry>
+        <mesh filename="package://mini_pupper_description/meshes/mini_pupper_2/lb3.stl" scale="1 1 1"/>
       </geometry>
     </collision>
@@ -291,12 +286,11 @@
       <origin xyz="-0.089299 0 0.015543" rpy="0 0 0"/>
       <geometry>
-        <mesh filename="file://$(find mini_pupper_description)/meshes/mini_pupper_2/Body_front.stl" scale="1 1 1"/>
-      </geometry>
-      <material name="opaque2552210"/>
+        <mesh filename="package://mini_pupper_description/meshes/mini_pupper_2/Body_front.dae" scale="1 1 1"/>
+      </geometry>
     </visual>
     <collision>
       <origin xyz="-0.089299 0 0.015543" rpy="0 0 0"/>
       <geometry>
-        <mesh filename="file://$(find mini_pupper_description)/meshes/mini_pupper_2/Body_front.stl" scale="1 1 1"/>
+        <mesh filename="package://mini_pupper_description/meshes/mini_pupper_2/Body_front.stl" scale="1 1 1"/>
       </geometry>
     </collision>
@@ -311,12 +305,11 @@
       <origin xyz="0.087701 0.023505 -0.026457" rpy="0 0 0"/>
       <geometry>
-        <mesh filename="file://$(find mini_pupper_description)/meshes/mini_pupper_2/Board_PCB.stl" scale="1 1 1"/>
-      </geometry>
-      <material name="opaque646464"/>
+        <mesh filename="package://mini_pupper_description/meshes/mini_pupper_2/Board_PCB.dae" scale="1 1 1"/>
+      </geometry>
     </visual>
     <collision>
       <origin xyz="0.087701 0.023505 -0.026457" rpy="0 0 0"/>
       <geometry>
-        <mesh filename="file://$(find mini_pupper_description)/meshes/mini_pupper_2/Board_PCB.stl" scale="1 1 1"/>
+        <mesh filename="package://mini_pupper_description/meshes/mini_pupper_2/Board_PCB.stl" scale="1 1 1"/>
       </geometry>
     </collision>
@@ -331,12 +324,11 @@
       <origin xyz="-0.061334 3.3e-05 -0.026457" rpy="0 0 0"/>
       <geometry>
-        <mesh filename="file://$(find mini_pupper_description)/meshes/mini_pupper_2/Board_connectors_1.stl" scale="1 1 1"/>
-      </geometry>
-      <material name="opaque2491590"/>
+        <mesh filename="package://mini_pupper_description/meshes/mini_pupper_2/Board_connectors_1.dae" scale="1 1 1"/>
+      </geometry>
     </visual>
     <collision>
       <origin xyz="-0.061334 3.3e-05 -0.026457" rpy="0 0 0"/>
       <geometry>
-        <mesh filename="file://$(find mini_pupper_description)/meshes/mini_pupper_2/Board_connectors_1.stl" scale="1 1 1"/>
+        <mesh filename="package://mini_pupper_description/meshes/mini_pupper_2/Board_connectors_1.stl" scale="1 1 1"/>
       </geometry>
     </collision>
@@ -351,12 +343,11 @@
       <origin xyz="0.045346 5e-06 -0.026457" rpy="0 0 0"/>
       <geometry>
-        <mesh filename="file://$(find mini_pupper_description)/meshes/mini_pupper_2/Board_connectors_2.stl" scale="1 1 1"/>
-      </geometry>
-      <material name="opaque255255255"/>
+        <mesh filename="package://mini_pupper_description/meshes/mini_pupper_2/Board_connectors_2.dae" scale="1 1 1"/>
+      </geometry>
     </visual>
     <collision>
       <origin xyz="0.045346 5e-06 -0.026457" rpy="0 0 0"/>
       <geometry>
-        <mesh filename="file://$(find mini_pupper_description)/meshes/mini_pupper_2/Board_connectors_2.stl" scale="1 1 1"/>
+        <mesh filename="package://mini_pupper_description/meshes/mini_pupper_2/Board_connectors_2.stl" scale="1 1 1"/>
       </geometry>
     </collision>
@@ -381,9 +372,6 @@
       <geometry>
         <mesh
-          filename="file://$(find mini_pupper_description)/meshes/mini_pupper_2/lidar.stl" />
-      </geometry>
-      <material name="">
-        <color rgba="0.2 0.2 0.2 1" />
-      </material>
+          filename="package://mini_pupper_description/meshes/mini_pupper_2/lidar.dae" />
+      </geometry>
     </visual>
     <collision>
@@ -391,5 +379,5 @@
       <geometry>
         <mesh
-          filename="file://$(find mini_pupper_description)/meshes/mini_pupper_2/lidar.stl" />
+          filename="package://mini_pupper_description/meshes/mini_pupper_2/lidar.stl" />
       </geometry>
     </collision>
@@ -404,12 +392,11 @@
       <origin xyz="0 0 0" rpy="0 0 0"/>
       <geometry>
-        <mesh filename="file://$(find mini_pupper_description)/meshes/mini_pupper_2/rffoot.stl" scale="1 1 1"/>
-      </geometry>
-      <material name="opaque666666"/>
-    </visual>
-    <collision>
-      <origin xyz="0 0 0" rpy="0 0 0"/>
-      <geometry>
-        <mesh filename="file://$(find mini_pupper_description)/meshes/mini_pupper_2/rffoot.stl" scale="1 1 1"/>
+        <mesh filename="package://mini_pupper_description/meshes/mini_pupper_2/rffoot.dae" scale="1 1 1"/>
+      </geometry>
+    </visual>
+    <collision>
+      <origin xyz="0 0 0" rpy="0 0 0"/>
+      <geometry>
+        <mesh filename="package://mini_pupper_description/meshes/mini_pupper_2/rffoot.stl" scale="1 1 1"/>
       </geometry>
     </collision>
@@ -424,12 +411,11 @@
       <origin xyz="0 0 0" rpy="0 0 0"/>
       <geometry>
-        <mesh filename="file://$(find mini_pupper_description)/meshes/mini_pupper_2/rbfoot.stl" scale="1 1 1"/>
-      </geometry>
-      <material name="opaque666666"/>
-    </visual>
-    <collision>
-      <origin xyz="0 0 0" rpy="0 0 0"/>
-      <geometry>
-        <mesh filename="file://$(find mini_pupper_description)/meshes/mini_pupper_2/rbfoot.stl" scale="1 1 1"/>
+        <mesh filename="package://mini_pupper_description/meshes/mini_pupper_2/rbfoot.dae" scale="1 1 1"/>
+      </geometry>
+    </visual>
+    <collision>
+      <origin xyz="0 0 0" rpy="0 0 0"/>
+      <geometry>
+        <mesh filename="package://mini_pupper_description/meshes/mini_pupper_2/rbfoot.stl" scale="1 1 1"/>
       </geometry>
     </collision>
@@ -444,12 +430,11 @@
       <origin xyz="0 0 0" rpy="0 0 0"/>
       <geometry>
-        <mesh filename="file://$(find mini_pupper_description)/meshes/mini_pupper_2/lbfoot.stl" scale="1 1 1"/>
-      </geometry>
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
Commit message: cleanup

File: mini_pupper_description/urdf/mini_pupper_2/mini_pupper_description.urdf.xacro (robot description, xacro)
@@ -955,4 +955,13 @@
     <kp>100000.0</kp>
     <kd>1.0</kd>
+    <mu1>1.5</mu1>
+    <mu2>1.5</mu2>
+    <maxVel>0.0</maxVel>
+    <minDepth>0.001</minDepth>
+    <material>Gazebo/FlatBlack</material>
+  </gazebo>
+  <gazebo reference="rf1">
+    <kp>100000.0</kp>
+    <kd>1.0</kd>
     <mu1>0.8</mu1>
     <mu2>0.8</mu2>
@@ -961,5 +970,8 @@
     <material>Gazebo/FlatBlack</material>
   </gazebo>
-  <gazebo reference="rf1">
+  <gazebo reference="rpf1">
+    <material>Gazebo/Yellow</material>
+  </gazebo>
+  <gazebo reference="rf2">
     <kp>100000.0</kp>
     <kd>1.0</kd>
@@ -970,8 +982,8 @@
     <material>Gazebo/FlatBlack</material>
   </gazebo>
-  <gazebo reference="rpf1">
+  <gazebo reference="rpf2">
     <material>Gazebo/Yellow</material>
   </gazebo>
-  <gazebo reference="rf2">
+  <gazebo reference="rf3">
     <kp>100000.0</kp>
     <kd>1.0</kd>
@@ -982,8 +994,14 @@
     <material>Gazebo/FlatBlack</material>
   </gazebo>
-  <gazebo reference="rpf2">
-    <material>Gazebo/Yellow</material>
-  </gazebo>
-  <gazebo reference="rf3">
+  <gazebo reference="rffoot">
+    <kp>100000.0</kp>
+    <kd>1.0</kd>
+    <mu1>1.5</mu1>
+    <mu2>1.5</mu2>
+    <maxVel>0.0</maxVel>
+    <minDepth>0.001</minDepth>
+    <material>Gazebo/FlatBlack</material>
+  </gazebo>
+  <gazebo reference="lb1">
     <kp>100000.0</kp>
     <kd>1.0</kd>
@@ -994,5 +1012,8 @@
     <material>Gazebo/FlatBlack</material>
   </gazebo>
-  <gazebo reference="rffoot">
+  <gazebo reference="lpb1">
+    <material>Gazebo/Yellow</material>
+  </gazebo>
+  <gazebo reference="lb2">
     <kp>100000.0</kp>
     <kd>1.0</kd>
@@ -1003,5 +1024,8 @@
     <material>Gazebo/FlatBlack</material>
   </gazebo>
-  <gazebo reference="lb1">
+  <gazebo reference="lpb2">
+    <material>Gazebo/Yellow</material>
+  </gazebo>
+  <gazebo reference="lb3">
     <kp>100000.0</kp>
     <kd>1.0</kd>
@@ -1012,8 +1036,14 @@
     <material>Gazebo/FlatBlack</material>
   </gazebo>
-  <gazebo reference="lpb1">
-    <material>Gazebo/Yellow</material>
-  </gazebo>
-  <gazebo reference="lb2">
+  <gazebo reference="lbfoot">
+    <kp>100000.0</kp>
+    <kd>1.0</kd>
+    <mu1>1.5</mu1>
+    <mu2>1.5</mu2>
+    <maxVel>0.0</maxVel>
+    <minDepth>0.001</minDepth>
+    <material>Gazebo/FlatBlack</material>
+  </gazebo>
+  <gazebo reference="rb1">
     <kp>100000.0</kp>
     <kd>1.0</kd>
@@ -1024,8 +1054,8 @@
     <material>Gazebo/FlatBlack</material>
   </gazebo>
-  <gazebo reference="lpb2">
+  <gazebo reference="rpb1">
     <material>Gazebo/Yellow</material>
   </gazebo>
-  <gazebo reference="lb3">
+  <gazebo reference="rb2">
     <kp>100000.0</kp>
     <kd>1.0</kd>
@@ -1036,5 +1066,8 @@
     <material>Gazebo/FlatBlack</material>
   </gazebo>
-  <gazebo reference="lbfoot">
+  <gazebo reference="rpb2">
+    <material>Gazebo/Yellow</material>
+  </gazebo>
+  <gazebo reference="rb3">
     <kp>100000.0</kp>
     <kd>1.0</kd>
@@ -1045,42 +1078,9 @@
     <material>Gazebo/FlatBlack</material>
   </gazebo>
-  <gazebo reference="rb1">
-    <kp>100000.0</kp>
-    <kd>1.0</kd>
-    <mu1>0.8</mu1>
-    <mu2>0.8</mu2>
-    <maxVel>0.0</maxVel>
-    <minDepth>0.001</minDepth>
-    <material>Gazebo/FlatBlack</material>
-  </gazebo>
-  <gazebo reference="rpb1">
-    <material>Gazebo/Yellow</material>
-  </gazebo>
-  <gazebo reference="rb2">
-    <kp>100000.0</kp>
-    <kd>1.0</kd>
-    <mu1>0.8</mu1>
-    <mu2>0.8</mu2>
-    <maxVel>0.0</maxVel>
-    <minDepth>0.001</minDepth>
-    <material>Gazebo/FlatBlack</material>
-  </gazebo>
-  <gazebo reference="rpb2">
-    <material>Gazebo/Yellow</material>
-  </gazebo>
-  <gazebo reference="rb3">
-    <kp>100000.0</kp>
-    <kd>1.0</kd>
-    <mu1>0.8</mu1>
-    <mu2>0.8</mu2>
-    <maxVel>0.0</maxVel>
-    <minDepth>0.001</minDepth>
-    <material>Gazebo/FlatBlack</material>
-  </gazebo>
   <gazebo reference="rbfoot">
     <kp>100000.0</kp>
     <kd>1.0</kd>
-    <mu1>0.8</mu1>
-    <mu2>0.8</mu2>
+    <mu1>1.5</mu1>
+    <mu2>1.5</mu2>
     <maxVel>0.0</maxVel>
     <minDepth>0.001</minDepth>
@@ -1093,5 +1093,5 @@
       <update_rate>30</update_rate>
       <pose>0 0 0 0 0 0</pose>
-      <visualize>false</visualize>
+      <visualize>true</visualize>
       <ray>
         <scan>
