Commit message: gzweb differences

File: mini_pupper_description/urdf/mini_pupper_2/mini_pupper_description_og.urdf.xacro (robot description, xacro)
@@ -24,21 +24,14 @@
       <origin xyz="0 0 0" rpy="0 0 0"/>
       <geometry>
-        <mesh filename="package://mini_pupper_description/meshes/mini_pupper_2/base_link_black.dae" scale="1 1 1"/>
-      </geometry>
-    </visual>
-    <collision>
-      <origin xyz="0 0 0" rpy="0 0 0"/>
-      <geometry>
-        <mesh filename="package://mini_pupper_description/meshes/mini_pupper_2/base_link.stl" scale="1 1 1"/>
-      </geometry>
-    </collision>
-  </link>
-  <link name="display_link">
-    <visual>
-      <origin xyz="0 0 0" rpy="0 0 0"/>
-      <geometry>
-        <mesh filename="package://mini_pupper_description/meshes/mini_pupper_2/displayscreen.dae" scale="1 1 1"/>
-      </geometry>
-    </visual>
+        <mesh filename="file://$(find mini_pupper_description)/meshes/mini_pupper_2/base_link.stl" scale="1 1 1"/>
+      </geometry>
+      <material name="opaque252525"/>
+    </visual>
+    <collision>
+      <origin xyz="0 0 0" rpy="0 0 0"/>
+      <geometry>
+        <mesh filename="file://$(find mini_pupper_description)/meshes/mini_pupper_2/base_link.stl" scale="1 1 1"/>
+      </geometry>
+    </collision>
   </link>
   <link name="base_inertia">
@@ -58,11 +51,12 @@
       <origin xyz="0 0 0" rpy="0 0 0"/>
       <geometry>
-        <mesh filename="package://mini_pupper_description/meshes/mini_pupper_2/lf1_black.dae" scale="1 1 1"/>
-      </geometry>
-    </visual>
-    <collision>
-      <origin xyz="0 0 0" rpy="0 0 0"/>
-      <geometry>
-        <mesh filename="package://mini_pupper_description/meshes/mini_pupper_2/lf1.stl" scale="1 1 1"/>
+        <mesh filename="file://$(find mini_pupper_description)/meshes/mini_pupper_2/lf1.stl" scale="1 1 1"/>
+      </geometry>
+      <material name="opaque666666"/>
+    </visual>
+    <collision>
+      <origin xyz="0 0 0" rpy="0 0 0"/>
+      <geometry>
+        <mesh filename="file://$(find mini_pupper_description)/meshes/mini_pupper_2/lf1.stl" scale="1 1 1"/>
       </geometry>
     </collision>
@@ -77,11 +71,12 @@
       <origin xyz="0 0 0" rpy="0 0 0"/>
       <geometry>
-        <mesh filename="package://mini_pupper_description/meshes/mini_pupper_2/lf2.dae" scale="1 1 1"/>
-      </geometry>
-    </visual>
-    <collision>
-      <origin xyz="0 0 0" rpy="0 0 0"/>
-      <geometry>
-        <mesh filename="package://mini_pupper_description/meshes/mini_pupper_2/lf2.stl" scale="1 1 1"/>
+        <mesh filename="file://$(find mini_pupper_description)/meshes/mini_pupper_2/lf2.stl" scale="1 1 1"/>
+      </geometry>
+      <material name="opaque636363"/>
+    </visual>
+    <collision>
+      <origin xyz="0 0 0" rpy="0 0 0"/>
+      <geometry>
+        <mesh filename="file://$(find mini_pupper_description)/meshes/mini_pupper_2/lf2.stl" scale="1 1 1"/>
       </geometry>
     </collision>
@@ -96,11 +91,12 @@
       <origin xyz="0 0 0" rpy="0 0 0"/>
       <geometry>
-        <mesh filename="package://mini_pupper_description/meshes/mini_pupper_2/lf3.dae" scale="1 1 1"/>
-      </geometry>
-    </visual>
-    <collision>
-      <origin xyz="0 0 0" rpy="0 0 0"/>
-      <geometry>
-        <mesh filename="package://mini_pupper_description/meshes/mini_pupper_2/lf3.stl" scale="1 1 1"/>
+        <mesh filename="file://$(find mini_pupper_description)/meshes/mini_pupper_2/lf3.stl" scale="1 1 1"/>
+      </geometry>
+      <material name="opaque252525"/>
+    </visual>
+    <collision>
+      <origin xyz="0 0 0" rpy="0 0 0"/>
+      <geometry>
+        <mesh filename="file://$(find mini_pupper_description)/meshes/mini_pupper_2/lf3.stl" scale="1 1 1"/>
       </geometry>
     </collision>
@@ -115,11 +111,12 @@
       <origin xyz="0 0 0" rpy="0 0 0"/>
       <geometry>
-        <mesh filename="package://mini_pupper_description/meshes/mini_pupper_2/rf1.dae" scale="1 1 1"/>
-      </geometry>
-    </visual>
-    <collision>
-      <origin xyz="0 0 0" rpy="0 0 0"/>
-      <geometry>
-        <mesh filename="package://mini_pupper_description/meshes/mini_pupper_2/rf1.stl" scale="1 1 1"/>
+        <mesh filename="file://$(find mini_pupper_description)/meshes/mini_pupper_2/rf1.stl" scale="1 1 1"/>
+      </geometry>
+      <material name="opaque666666"/>
+    </visual>
+    <collision>
+      <origin xyz="0 0 0" rpy="0 0 0"/>
+      <geometry>
+        <mesh filename="file://$(find mini_pupper_description)/meshes/mini_pupper_2/rf1.stl" scale="1 1 1"/>
       </geometry>
     </collision>
@@ -134,11 +131,12 @@
       <origin xyz="0 0 0" rpy="0 0 0"/>
       <geometry>
-        <mesh filename="package://mini_pupper_description/meshes/mini_pupper_2/rf2.dae" scale="1 1 1"/>
-      </geometry>
-    </visual>
-    <collision>
-      <origin xyz="0 0 0" rpy="0 0 0"/>
-      <geometry>
-        <mesh filename="package://mini_pupper_description/meshes/mini_pupper_2/rf2.stl" scale="1 1 1"/>
+        <mesh filename="file://$(find mini_pupper_description)/meshes/mini_pupper_2/rf2.stl" scale="1 1 1"/>
+      </geometry>
+      <material name="opaque636363"/>
+    </visual>
+    <collision>
+      <origin xyz="0 0 0" rpy="0 0 0"/>
+      <geometry>
+        <mesh filename="file://$(find mini_pupper_description)/meshes/mini_pupper_2/rf2.stl" scale="1 1 1"/>
       </geometry>
     </collision>
@@ -153,11 +151,12 @@
       <origin xyz="0 0 0" rpy="0 0 0"/>
       <geometry>
-        <mesh filename="package://mini_pupper_description/meshes/mini_pupper_2/rf3_black.dae" scale="1 1 1"/>
-      </geometry>
-    </visual>
-    <collision>
-      <origin xyz="0 0 0" rpy="0 0 0"/>
-      <geometry>
-        <mesh filename="package://mini_pupper_description/meshes/mini_pupper_2/rf3.stl" scale="1 1 1"/>
+        <mesh filename="file://$(find mini_pupper_description)/meshes/mini_pupper_2/rf3.stl" scale="1 1 1"/>
+      </geometry>
+      <material name="opaque252525"/>
+    </visual>
+    <collision>
+      <origin xyz="0 0 0" rpy="0 0 0"/>
+      <geometry>
+        <mesh filename="file://$(find mini_pupper_description)/meshes/mini_pupper_2/rf3.stl" scale="1 1 1"/>
       </geometry>
     </collision>
@@ -172,11 +171,12 @@
       <origin xyz="0 0 0" rpy="0 0 0"/>
       <geometry>
-        <mesh filename="package://mini_pupper_description/meshes/mini_pupper_2/rb1.dae" scale="1 1 1"/>
-      </geometry>
-    </visual>
-    <collision>
-      <origin xyz="0 0 0" rpy="0 0 0"/>
-      <geometry>
-        <mesh filename="package://mini_pupper_description/meshes/mini_pupper_2/rb1.stl" scale="1 1 1"/>
+        <mesh filename="file://$(find mini_pupper_description)/meshes/mini_pupper_2/rb1.stl" scale="1 1 1"/>
+      </geometry>
+      <material name="opaque666666"/>
+    </visual>
+    <collision>
+      <origin xyz="0 0 0" rpy="0 0 0"/>
+      <geometry>
+        <mesh filename="file://$(find mini_pupper_description)/meshes/mini_pupper_2/rb1.stl" scale="1 1 1"/>
       </geometry>
     </collision>
@@ -191,11 +191,12 @@
       <origin xyz="0 0 0" rpy="0 0 0"/>
       <geometry>
-        <mesh filename="package://mini_pupper_description/meshes/mini_pupper_2/rb2.dae" scale="1 1 1"/>
-      </geometry>
-    </visual>
-    <collision>
-      <origin xyz="0 0 0" rpy="0 0 0"/>
-      <geometry>
-        <mesh filename="package://mini_pupper_description/meshes/mini_pupper_2/rb2.stl" scale="1 1 1"/>
+        <mesh filename="file://$(find mini_pupper_description)/meshes/mini_pupper_2/rb2.stl" scale="1 1 1"/>
+      </geometry>
+      <material name="opaque636363"/>
+    </visual>
+    <collision>
+      <origin xyz="0 0 0" rpy="0 0 0"/>
+      <geometry>
+        <mesh filename="file://$(find mini_pupper_description)/meshes/mini_pupper_2/rb2.stl" scale="1 1 1"/>
       </geometry>
     </collision>
@@ -210,11 +211,12 @@
       <origin xyz="0 0 0" rpy="0 0 0"/>
       <geometry>
-        <mesh filename="package://mini_pupper_description/meshes/mini_pupper_2/rb3.dae" scale="1 1 1"/>
-      </geometry>
-    </visual>
-    <collision>
-      <origin xyz="0 0 0" rpy="0 0 0"/>
-      <geometry>
-        <mesh filename="package://mini_pupper_description/meshes/mini_pupper_2/rb3.stl" scale="1 1 1"/>
+        <mesh filename="file://$(find mini_pupper_description)/meshes/mini_pupper_2/rb3.stl" scale="1 1 1"/>
+      </geometry>
+      <material name="opaque252525"/>
+    </visual>
+    <collision>
+      <origin xyz="0 0 0" rpy="0 0 0"/>
+      <geometry>
+        <mesh filename="file://$(find mini_pupper_description)/meshes/mini_pupper_2/rb3.stl" scale="1 1 1"/>
       </geometry>
     </collision>
@@ -229,11 +231,12 @@
       <origin xyz="0 0 0" rpy="0 0 0"/>
       <geometry>
-        <mesh filename="package://mini_pupper_description/meshes/mini_pupper_2/lb1.dae" scale="1 1 1"/>
-      </geometry>
-    </visual>
-    <collision>
-      <origin xyz="0 0 0" rpy="0 0 0"/>
-      <geometry>
-        <mesh filename="package://mini_pupper_description/meshes/mini_pupper_2/lb1.stl" scale="1 1 1"/>
+        <mesh filename="file://$(find mini_pupper_description)/meshes/mini_pupper_2/lb1.stl" scale="1 1 1"/>
+      </geometry>
+      <material name="opaque666666"/>
+    </visual>
+    <collision>
+      <origin xyz="0 0 0" rpy="0 0 0"/>
+      <geometry>
+        <mesh filename="file://$(find mini_pupper_description)/meshes/mini_pupper_2/lb1.stl" scale="1 1 1"/>
       </geometry>
     </collision>
@@ -248,11 +251,12 @@
       <origin xyz="0 0 0" rpy="0 0 0"/>
       <geometry>
-        <mesh filename="package://mini_pupper_description/meshes/mini_pupper_2/lb2.dae" scale="1 1 1"/>
-      </geometry>
-    </visual>
-    <collision>
-      <origin xyz="0 0 0" rpy="0 0 0"/>
-      <geometry>
-        <mesh filename="package://mini_pupper_description/meshes/mini_pupper_2/lb2.stl" scale="1 1 1"/>
+        <mesh filename="file://$(find mini_pupper_description)/meshes/mini_pupper_2/lb2.stl" scale="1 1 1"/>
+      </geometry>
+      <material name="opaque636363"/>
+    </visual>
+    <collision>
+      <origin xyz="0 0 0" rpy="0 0 0"/>
+      <geometry>
+        <mesh filename="file://$(find mini_pupper_description)/meshes/mini_pupper_2/lb2.stl" scale="1 1 1"/>
       </geometry>
     </collision>
@@ -267,11 +271,12 @@
       <origin xyz="0 0 0" rpy="0 0 0"/>
       <geometry>
-        <mesh filename="package://mini_pupper_description/meshes/mini_pupper_2/lb3.dae" scale="1 1 1"/>
-      </geometry>
-    </visual>
-    <collision>
-      <origin xyz="0 0 0" rpy="0 0 0"/>
-      <geometry>
-        <mesh filename="package://mini_pupper_description/meshes/mini_pupper_2/lb3.stl" scale="1 1 1"/>
+        <mesh filename="file://$(find mini_pupper_description)/meshes/mini_pupper_2/lb3.stl" scale="1 1 1"/>
+      </geometry>
+      <material name="opaque252525"/>
+    </visual>
+    <collision>
+      <origin xyz="0 0 0" rpy="0 0 0"/>
+      <geometry>
+        <mesh filename="file://$(find mini_pupper_description)/meshes/mini_pupper_2/lb3.stl" scale="1 1 1"/>
       </geometry>
     </collision>
@@ -286,11 +291,12 @@
       <origin xyz="-0.089299 0 0.015543" rpy="0 0 0"/>
       <geometry>
-        <mesh filename="package://mini_pupper_description/meshes/mini_pupper_2/Body_front.dae" scale="1 1 1"/>
-      </geometry>
+        <mesh filename="file://$(find mini_pupper_description)/meshes/mini_pupper_2/Body_front.stl" scale="1 1 1"/>
+      </geometry>
+      <material name="opaque2552210"/>
     </visual>
     <collision>
       <origin xyz="-0.089299 0 0.015543" rpy="0 0 0"/>
       <geometry>
-        <mesh filename="package://mini_pupper_description/meshes/mini_pupper_2/Body_front.stl" scale="1 1 1"/>
+        <mesh filename="file://$(find mini_pupper_description)/meshes/mini_pupper_2/Body_front.stl" scale="1 1 1"/>
       </geometry>
     </collision>
@@ -305,11 +311,12 @@
       <origin xyz="0.087701 0.023505 -0.026457" rpy="0 0 0"/>
       <geometry>
-        <mesh filename="package://mini_pupper_description/meshes/mini_pupper_2/Board_PCB.dae" scale="1 1 1"/>
-      </geometry>
+        <mesh filename="file://$(find mini_pupper_description)/meshes/mini_pupper_2/Board_PCB.stl" scale="1 1 1"/>
+      </geometry>
+      <material name="opaque646464"/>
     </visual>
     <collision>
       <origin xyz="0.087701 0.023505 -0.026457" rpy="0 0 0"/>
       <geometry>
-        <mesh filename="package://mini_pupper_description/meshes/mini_pupper_2/Board_PCB.stl" scale="1 1 1"/>
+        <mesh filename="file://$(find mini_pupper_description)/meshes/mini_pupper_2/Board_PCB.stl" scale="1 1 1"/>
       </geometry>
     </collision>
@@ -324,11 +331,12 @@
       <origin xyz="-0.061334 3.3e-05 -0.026457" rpy="0 0 0"/>
       <geometry>
-        <mesh filename="package://mini_pupper_description/meshes/mini_pupper_2/Board_connectors_1.dae" scale="1 1 1"/>
-      </geometry>
+        <mesh filename="file://$(find mini_pupper_description)/meshes/mini_pupper_2/Board_connectors_1.stl" scale="1 1 1"/>
+      </geometry>
+      <material name="opaque2491590"/>
     </visual>
     <collision>
       <origin xyz="-0.061334 3.3e-05 -0.026457" rpy="0 0 0"/>
       <geometry>
-        <mesh filename="package://mini_pupper_description/meshes/mini_pupper_2/Board_connectors_1.stl" scale="1 1 1"/>
+        <mesh filename="file://$(find mini_pupper_description)/meshes/mini_pupper_2/Board_connectors_1.stl" scale="1 1 1"/>
       </geometry>
     </collision>
@@ -343,11 +351,12 @@
       <origin xyz="0.045346 5e-06 -0.026457" rpy="0 0 0"/>
       <geometry>
-        <mesh filename="package://mini_pupper_description/meshes/mini_pupper_2/Board_connectors_2.dae" scale="1 1 1"/>
-      </geometry>
+        <mesh filename="file://$(find mini_pupper_description)/meshes/mini_pupper_2/Board_connectors_2.stl" scale="1 1 1"/>
+      </geometry>
+      <material name="opaque255255255"/>
     </visual>
     <collision>
       <origin xyz="0.045346 5e-06 -0.026457" rpy="0 0 0"/>
       <geometry>
-        <mesh filename="package://mini_pupper_description/meshes/mini_pupper_2/Board_connectors_2.stl" scale="1 1 1"/>
+        <mesh filename="file://$(find mini_pupper_description)/meshes/mini_pupper_2/Board_connectors_2.stl" scale="1 1 1"/>
       </geometry>
     </collision>
@@ -372,6 +381,9 @@
       <geometry>
         <mesh
-          filename="package://mini_pupper_description/meshes/mini_pupper_2/lidar.dae" />
-      </geometry>
+          filename="file://$(find mini_pupper_description)/meshes/mini_pupper_2/lidar.stl" />
+      </geometry>
+      <material name="">
+        <color rgba="0.2 0.2 0.2 1" />
+      </material>
     </visual>
     <collision>
@@ -379,5 +391,5 @@
       <geometry>
         <mesh
-          filename="package://mini_pupper_description/meshes/mini_pupper_2/lidar.stl" />
+          filename="file://$(find mini_pupper_description)/meshes/mini_pupper_2/lidar.stl" />
       </geometry>
     </collision>
@@ -392,11 +404,12 @@
       <origin xyz="0 0 0" rpy="0 0 0"/>
       <geometry>
-        <mesh filename="package://mini_pupper_description/meshes/mini_pupper_2/rffoot.dae" scale="1 1 1"/>
-      </geometry>
-    </visual>
-    <collision>
-      <origin xyz="0 0 0" rpy="0 0 0"/>
-      <geometry>
-        <mesh filename="package://mini_pupper_description/meshes/mini_pupper_2/rffoot.stl" scale="1 1 1"/>
+        <mesh filename="file://$(find mini_pupper_description)/meshes/mini_pupper_2/rffoot.stl" scale="1 1 1"/>
+      </geometry>
+      <material name="opaque666666"/>
+    </visual>
+    <collision>
+      <origin xyz="0 0 0" rpy="0 0 0"/>
+      <geometry>
+        <mesh filename="file://$(find mini_pupper_description)/meshes/mini_pupper_2/rffoot.stl" scale="1 1 1"/>
       </geometry>
     </collision>
@@ -411,11 +424,12 @@
       <origin xyz="0 0 0" rpy="0 0 0"/>
       <geometry>
-        <mesh filename="package://mini_pupper_description/meshes/mini_pupper_2/rbfoot.dae" scale="1 1 1"/>
-      </geometry>
-    </visual>
-    <collision>
-      <origin xyz="0 0 0" rpy="0 0 0"/>
-      <geometry>
-        <mesh filename="package://mini_pupper_description/meshes/mini_pupper_2/rbfoot.stl" scale="1 1 1"/>
+        <mesh filename="file://$(find mini_pupper_description)/meshes/mini_pupper_2/rbfoot.stl" scale="1 1 1"/>
+      </geometry>
+      <material name="opaque666666"/>
+    </visual>
+    <collision>
+      <origin xyz="0 0 0" rpy="0 0 0"/>
+      <geometry>
+        <mesh filename="file://$(find mini_pupper_description)/meshes/mini_pupper_2/rbfoot.stl" scale="1 1 1"/>
       </geometry>
     </collision>
@@ -430,11 +444,12 @@
       <origin xyz="0 0 0" rpy="0 0 0"/>
       <geometry>
-        <mesh filename="package://mini_pupper_description/meshes/mini_pupper_2/lbfoot.dae" scale="1 1 1"/>
-      </geometry>
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